Commit message: changed joints' names to panda_jointX and fixed visualization

File: franka_coppelia_hw/urdf/panda.urdf (robot description, URDF)
Before this commit: robot Franka, 8 links, 7 joints
Joints:
- removed joint joint0
- removed joint joint1
- removed joint joint2
- removed joint joint3
- removed joint joint4
- removed joint joint5
- removed joint joint6
- added joint panda_joint0: type revolute, parent robot_base, child link2resp, origin xyz=-0.249729 -0.074988 0.000000 rpy=-3.141593 3.141593 -3.141593, axis 0 0 1, limit lower=-2.8972465991974 upper=2.8972465991974 effort=87.0 velocity=2.1749997138977
- added joint panda_joint1: type revolute, parent link2resp, child link3resp, origin xyz=-0.000000 -0.000000 0.333000 rpy=1.570796 3.141593 3.141593, axis 0 0 1, limit lower=-1.7627825737 upper=1.7627825737 effort=87.0 velocity=2.1749997138977
- added joint panda_joint2: type revolute, parent link3resp, child link4resp, origin xyz=-0.000000 0.000000 0.000000 rpy=-1.570797 3.141593 -3.141593, axis 0 0 1, limit lower=-2.8972465991974 upper=2.8972465991974 effort=87.0 velocity=2.1749997138977
- added joint panda_joint3: type revolute, parent link4resp, child link5resp, origin xyz=0.082500 -0.000000 0.316000 rpy=-1.570796 3.141593 -3.141592, axis 0 0 1, limit lower=-3.0019662380219 upper=0.0 effort=87.0 velocity=2.1749997138977
- added joint panda_joint4: type revolute, parent link5resp, child link6resp, origin xyz=-0.055513 0.388820 -0.000000 rpy=1.570796 3.141593 3.071779, axis 0 0 1, limit lower=-2.8972465991974 upper=2.8972465991974 effort=12.0 velocity=2.610000371933
- added joint panda_joint5: type revolute, parent link6resp, child link7resp, origin xyz=-0.000000 -0.000000 0.000000 rpy=-1.570796 3.141593 -3.141593, axis 0 0 1, limit lower=-0.017453292384744 upper=3.7524577584118 effort=12.0 velocity=2.610000371933
- added joint panda_joint6: type revolute, parent link7resp, child link8resp, origin xyz=0.088000 0.000000 -0.000000 rpy=-1.570796 3.141592 3.141593, axis 0 0 1, limit lower=-2.8972465991974 upper=2.8972465991974 effort=12.0 velocity=2.610000371933

Commit message: debug

File: franka_coppelia_hw/urdf/panda.urdf (robot description, URDF)
Before this commit: robot Franka, 8 links, 7 joints
Joints:
- removed joint panda_joint0
- added joint panda_joint7: type revolute, parent link7resp, child link8resp, origin xyz=0.088000 0.000000 -0.000000 rpy=-1.570796 3.141592 3.141593, axis 0 0 1, limit lower=-2.8972465991974 upper=2.8972465991974 effort=12.0 velocity=2.610000371933
- joint panda_joint1: child link3resp -> link2resp; limit lower=-1.7627825737 upper=1.7627825737 effort=87.0 velocity=2.1749997138977 -> lower=-2.8972465991974 upper=2.8972465991974 effort=87.0 velocity=2.1749997138977; origin xyz=-0.000000 -0.000000 0.333000 rpy=1.570796 3.141593 3.141593 -> xyz=-0.249729 -0.074988 0.000000 rpy=-3.141593 3.141593 -3.141593; parent link2resp -> robot_base
- joint panda_joint2: child link4resp -> link3resp; limit lower=-2.8972465991974 upper=2.8972465991974 effort=87.0 velocity=2.1749997138977 -> lower=-1.7627825737 upper=1.7627825737 effort=87.0 velocity=2.1749997138977; origin xyz=-0.000000 0.000000 0.000000 rpy=-1.570797 3.141593 -3.141593 -> xyz=-0.000000 -0.000000 0.333000 rpy=1.570796 3.141593 3.141593; parent link3resp -> link2resp
- joint panda_joint3: child link5resp -> link4resp; limit lower=-3.0019662380219 upper=0.0 effort=87.0 velocity=2.1749997138977 -> lower=-2.8972465991974 upper=2.8972465991974 effort=87.0 velocity=2.1749997138977; origin xyz=0.082500 -0.000000 0.316000 rpy=-1.570796 3.141593 -3.141592 -> xyz=-0.000000 0.000000 0.000000 rpy=-1.570797 3.141593 -3.141593; parent link4resp -> link3resp
- joint panda_joint4: child link6resp -> link5resp; limit lower=-2.8972465991974 upper=2.8972465991974 effort=12.0 velocity=2.610000371933 -> lower=-3.0019662380219 upper=0.0 effort=87.0 velocity=2.1749997138977; origin xyz=-0.055513 0.388820 -0.000000 rpy=1.570796 3.141593 3.071779 -> xyz=0.082500 -0.000000 0.316000 rpy=-1.570796 3.141593 -3.141592; parent link5resp -> link4resp
- joint panda_joint5: child link7resp -> link6resp; limit lower=-0.017453292384744 upper=3.7524577584118 effort=12.0 velocity=2.610000371933 -> lower=-2.8972465991974 upper=2.8972465991974 effort=12.0 velocity=2.610000371933; origin xyz=-0.000000 -0.000000 0.000000 rpy=-1.570796 3.141593 -3.141593 -> xyz=-0.055513 0.388820 -0.000000 rpy=1.570796 3.141593 3.071779; parent link6resp -> link5resp
- joint panda_joint6: child link8resp -> link7resp; limit lower=-2.8972465991974 upper=2.8972465991974 effort=12.0 velocity=2.610000371933 -> lower=-0.017453292384744 upper=3.7524577584118 effort=12.0 velocity=2.610000371933; origin xyz=0.088000 0.000000 -0.000000 rpy=-1.570796 3.141592 3.141593 -> xyz=-0.000000 -0.000000 0.000000 rpy=-1.570796 3.141593 -3.141593; parent link7resp -> link6resp

File: franka_coppelia_hw/urdf/panda_arm.ros2_control.xacro (robot description, xacro)
@@ -20,5 +20,4 @@
           <state_interface name="position"/>
           <state_interface name="velocity"/>
-          <state_interface name="effort"/>
         </joint>
       </xacro:macro>
