Commit message: more debug

File: franka_coppelia_hw/urdf/panda_arm.xacro (robot description, xacro)
@@ -70,4 +70,9 @@
     </joint>
     <link name="${arm_id}_link2">
+      <inertial>
+            <origin xyz="0.000027 -0.031145 0.262891" rpy="-3.141593 3.141593 -3.141593" />
+            <inertia ixx="0.23965416449794" iyz="0.046543293301451" ixz="1.3128335716866e-05" ixy="1.8036869099987e-05" izz="0.096472146190744" iyy="0.20795149177852" />
+            <mass value="4.9706840515137" />
+      </inertial>
       <visual>
         <geometry>
@@ -103,4 +108,9 @@
     </joint>
     <link name="${arm_id}_link3">
+     <inertial>
+            <origin xyz="0.000012 -0.070031 0.031073" rpy="-1.570796 3.141593 -3.141593" />
+            <inertia ixx="0.021097005907894" iyz="0.0040788476591549" ixz="-9.6899135443004e-07" ixy="4.6746993616892e-06" izz="0.0083947222563338" iyy="0.018332235221749" />
+            <mass value="0.64692598581314" />
+      </inertial>
       <visual>
         <geometry>
@@ -136,4 +146,9 @@
     </joint>
     <link name="${arm_id}_link4">
+      <inertial>
+            <origin xyz="0.044418 0.025018 0.276461" rpy="-3.141592 3.141593 3.141593" />
+            <inertia ixx="0.037043165158734" iyz="-0.0066345366154784" ixz="-0.012283585683442" ixy="-0.0071662360347711" izz="0.037313700213202" iyy="0.044600332011806" />
+            <mass value="3.2286040782928" />
+      </inertial>
       <visual>
         <geometry>
@@ -169,4 +184,9 @@
     </joint>
     <link name="${arm_id}_link5">
+      <inertial>
+            <origin xyz="-0.036035 0.041072 0.024354" rpy="1.570796 3.141593 3.071779" />
+            <inertia ixx="0.04844892193307" iyz="-0.0086501440884625" ixz="0.016026606898086" ixy="0.0091601974989418" izz="0.047764716548773" iyy="0.05816570900911" />
+            <mass value="3.5878949165344" />
+      </inertial>
       <visual>
         <geometry>
@@ -220,4 +240,9 @@
     </joint>
     <link name="${arm_id}_link6">
+      <inertial>
+          <origin xyz="0.000101 0.038651 -0.110916" rpy="3.141593 3.141592 3.141592" />
+          <inertia ixx="0.03988537400492" iyz="-0.0078141474579038" ixz="-2.672442414716e-05" ixy="6.5734913571839e-07" izz="0.010430599214868" iyy="0.036230106859883" />
+          <mass value="1.2259459495544" />
+      </inertial>
       <visual>
         <geometry>
@@ -253,4 +278,9 @@
     </joint>
     <link name="${arm_id}_link7">
+      <inertial>
+          <origin xyz="0.050819 0.005558 0.005395" rpy="1.570796 3.141593 3.141593" />
+          <inertia ixx="0.0046587251169735" iyz="-6.1476550160376e-05" ixz="-0.00030740988325929" ixy="-0.00057744119112155" izz="0.0070729035771789" iyy="0.008643924526682" />
+          <mass value="1.6665550470352" />
+      </inertial>
       <visual>
         <geometry>
@@ -286,4 +316,9 @@
     </joint>
     <link name="${arm_id}_link8">
+      <inertial>
+            <origin xyz="-0.000077 -0.000876 0.078618" rpy="-0.000000 3.141593 -3.141592" />
+            <inertia ixx="0.0088670116631003" iyz="-9.1760218741593e-08" ixz="7.00227187462e-07" ixy="7.6321250755392e-11" izz="0.01180331651387" iyy="0.0088670122123097" />
+            <mass value="0.73552197217941" />
+      </inertial>
       <collision>
         <origin xyz="0.0424 0.0424 -0.0250" rpy="${pi} ${pi/2} ${pi/2}"/>

File: franka_coppelia_hw/urdf/test.xacro (robot description, xacro)
@@ -5,8 +5,5 @@
       <hardware>
         <xacro:if value="${use_fake_hardware}">
-          <plugin>franka_coppelia_hw/FrankaEffortHardware</plugin>
-          <param name="example_param_hw_start_duration_sec">0</param>
-          <param name="example_param_hw_stop_duration_sec">3.0</param>
-          <param name="example_param_hw_slowdown">100</param>
+          <plugin>fake_components/GenericSystem</plugin>
           <param name="fake_sensor_commands">${fake_sensor_commands}</param>
           <param name="state_following_offset">0.0</param>
@@ -19,14 +16,10 @@
       <xacro:macro name="configure_joint" params="joint_name initial_position initial_velocity initial_effort">
         <joint name="${joint_name}">
+          <param name="initial_position">${initial_position}</param>
+          <param name="initial_velocity">${initial_velocity}</param>
+          <param name="initial_effort">${initial_effort}</param>
           <command_interface name="effort"/>
-          <state_interface name="position">
-            <param name="initial_position">${initial_position}</param>
-          </state_interface>
-          <state_interface name="velocity">
-            <param name="initial_velocity">${initial_velocity}</param>
-          </state_interface>
-          <state_interface name="effort">
-            <param name="initial_effort">${initial_effort}</param>
-          </state_interface>
+          <state_interface name="position"/>
+          <state_interface name="velocity"/>
         </joint>
       </xacro:macro>
